File: Kicad/simple-midi-controller.kicad_pcb (KiCad board)
At the start: 2 copper layers, 70 x 50 mm, 14 parts, among them J1 Conn_02x06_Odd_Even, J2 Conn_01x03, J3 Conn_02x06_Odd_Even, J4 Conn_01x04, U1 MAX7219

Commit message: updated pcb design
Parts:
- R1: value R -> 150
Changed lines of the file:
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@@
 			)
 		)
-		(property "Value" "R"
-			(at 5.08 2.37 90)
-			(layer "F.Fab")
+		(property "Value" "150"
+			(at 5.08 0.06 90)
+			(layer "F.SilkS")
 			(effects
 				(font
 					(size 1 1)
-					(thickness 0.15)
+					(thickness 0.2)
+					(bold yes)
 				)
 			)
