File: Kicad/simple-midi-controller.kicad_sch (KiCad schematic)
At the start: 13 parts, among them J1 Conn_02x06_Odd_Even, J2 Conn_01x03, J3 Conn_02x06_Odd_Even, J4 Conn_01x04, U1 MAX7219

Commit message: updated pcb design
Parts:
- R1: value R -> 150
Changed lines of the file:
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@@
 			)
 		)
-		(property "Value" "R"
+		(property "Value" "150"
 			(at 92.71 106.68 90)
 			(effects
@@
 		(at 203.2 46.99 0)
 		(unit 1)
-		(exclude_from_sim no)
+		(exclude_from_sim yes)
 		(in_bom yes)
 		(on_board yes)
@@
 			(at 203.2 46.99 0)
 			(effects
-				(font
-					(size 1.27 1.27)
-				)
-				(hide yes)
-			)
-		)
-		(property "Sim.Enable" "0"
-			(at 203.2 46.99 0)
-			(effects
